Commit message: to be tested code

File: vehicle_common/urdf/vehicle_description.xacro (robot description, xacro)
@@ -15,15 +15,15 @@
     <child link="gps_link" />
   </joint>
-  <link name="zed2i_base_link"/>
+  <link name="zed_camera"/>
   <joint name="zed_camera_link" type="fixed">
     <origin xyz="2.8 0 0.5" rpy="0 0 0" />
     <parent link="base_link" />
-    <child link="zed2i_base_link" />
+    <child link="zed_camera" />
   </joint>
-  <link name="rs_lidar"/>
+  <link name="rslidar"/>
   <joint name="lidar_link" type="fixed">
     <origin xyz="2.8 0 0.2" rpy="0 0 0" />
     <parent link="base_link" />
-    <child link="rs_lidar" />
+    <child link="rslidar" />
   </joint>
 </robot>

Commit message: refactor: vehicle URDF to take from config file - Added config file for porter and half cabins - sensor locations are also to be taken from config file - sensor location details and vehicle dimentions are are in sync with master parameters - changed speed limis to motion_limits,  changed in corresponding nodes as well. - closes #189

File: vehicle_common/urdf/vehicle_description.xacro (robot description, xacro)
@@ -1,27 +1,47 @@
 <?xml version="1.0"?>
 <robot name="boson_vehicle" xmlns:xacro="http://ros.org/wiki/xacro">
+  <xacro:arg name="config_file" default="$(find vehicle_common)/params/half_cabin_config.yaml"/>
+  <xacro:property name="config_file_property" value = "$(arg config_file)"/>
   <xacro:property name="M_PI"     value="3.1415926535897931" />
-  <xacro:property name="yaml_file" value="$(find vehicle_common)/params/vehicle_config.yaml" />
-  <xacro:property name="vehicle_data" value="${load_yaml(yaml_file)}"/>
-<!--  <xacro:property name="val1" value="${props['val1']}" />-->
-<!--  <xacro:property name="gps_link_origin_xyz" value="${vehicle_data['fcu']['orientation'][0]} ${vehicle_data['fcu']['orientation'][1]} ${vehicle_data['fcu']['orientation'][2]}" />-->
-<!--  <xacro:property name="gps_link_origin_rpy" value="${vehicle_data['fcu']['orientation']}" />-->
-<!--  <xacro:property name="gps_link" value="${vehicle_data['robot_origin_frame']} " />-->
+  <xacro:property name="vehicle_info" value="${xacro.load_yaml(config_file_property)}"/>
   <link name="base_link"/>
   <link name="gps_link"/>
   <joint name="gps_joint" type="fixed">
-    <origin xyz="2 0 0.1" rpy="0 0 0" />
+    <origin
+        xyz="${vehicle_info['base_link']['gps_link']['x']}
+             ${vehicle_info['base_link']['gps_link']['y']}
+             ${vehicle_info['base_link']['gps_link']['z']}"
+        rpy="${vehicle_info['base_link']['gps_link']['roll']}
+             ${vehicle_info['base_link']['gps_link']['pitch']}
+             ${vehicle_info['base_link']['gps_link']['yaw']}"
+    />
     <parent link="base_link" />
     <child link="gps_link" />
   </joint>
-  <link name="zed_camera"/>
+  <link name="zed2i_base_link"/>
   <joint name="zed_camera_link" type="fixed">
-    <origin xyz="2.8 0 0.5" rpy="0 0 0" />
+    <!-- <origin xyz="2.8 0 0.5" rpy="0 0 0" /> -->
+    <origin
+        xyz="${vehicle_info['base_link']['zed2i_base_link']['x']}
+             ${vehicle_info['base_link']['zed2i_base_link']['y']}
+             ${vehicle_info['base_link']['zed2i_base_link']['z']}"
+        rpy="${vehicle_info['base_link']['zed2i_base_link']['roll']}
+             ${vehicle_info['base_link']['zed2i_base_link']['pitch']}
+             ${vehicle_info['base_link']['zed2i_base_link']['yaw']}"
+    />
     <parent link="base_link" />
-    <child link="zed_camera" />
+    <child link="zed2i_base_link" />
   </joint>
   <link name="rslidar"/>
   <joint name="3d_lidar_link" type="fixed">
-    <origin xyz="2.8 0 0.2" rpy="0 0 0" />
+    <!-- <origin xyz="2.8 0 0.2" rpy="0 0 0" /> -->
+    <origin
+        xyz="${vehicle_info['base_link']['rslidar']['x']}
+             ${vehicle_info['base_link']['rslidar']['y']}
+             ${vehicle_info['base_link']['rslidar']['z']}"
+        rpy="${vehicle_info['base_link']['rslidar']['roll']}
+             ${vehicle_info['base_link']['rslidar']['pitch']}
+             ${vehicle_info['base_link']['rslidar']['yaw']}"
+    />
     <parent link="base_link" />
     <child link="rslidar" />
@@ -29,5 +49,13 @@
   <link name="rplidar"/>
   <joint name="2d_lidar_link" type="fixed">
-    <origin xyz="2.8 0 0.1" rpy="0 0 0" />
+    <!-- <origin xyz="2.8 0 0.1" rpy="0 0 0" /> -->
+    <origin
+        xyz="${vehicle_info['base_link']['rplidar']['x']}
+             ${vehicle_info['base_link']['rplidar']['y']}
+             ${vehicle_info['base_link']['rplidar']['z']}"
+        rpy="${vehicle_info['base_link']['rplidar']['roll']}
+             ${vehicle_info['base_link']['rplidar']['pitch']}
+             ${vehicle_info['base_link']['rplidar']['yaw']}"
+    />
     <parent link="base_link" />
     <child link="rplidar" />

Commit message: fix : changed zed2i_base_link to zed_cemera

File: vehicle_common/urdf/vehicle_description.xacro (robot description, xacro)
@@ -19,17 +19,17 @@
     <child link="gps_link" />
   </joint>
-  <link name="zed2i_base_link"/>
+  <link name="zed_camera"/>
   <joint name="zed_camera_link" type="fixed">
     <!-- <origin xyz="2.8 0 0.5" rpy="0 0 0" /> -->
     <origin
-        xyz="${vehicle_info['base_link']['zed2i_base_link']['x']}
-             ${vehicle_info['base_link']['zed2i_base_link']['y']}
-             ${vehicle_info['base_link']['zed2i_base_link']['z']}"
-        rpy="${vehicle_info['base_link']['zed2i_base_link']['roll']}
-             ${vehicle_info['base_link']['zed2i_base_link']['pitch']}
-             ${vehicle_info['base_link']['zed2i_base_link']['yaw']}"
+        xyz="${vehicle_info['base_link']['zed_camera']['x']}
+             ${vehicle_info['base_link']['zed_camera']['y']}
+             ${vehicle_info['base_link']['zed_camera']['z']}"
+        rpy="${vehicle_info['base_link']['zed_camera']['roll']}
+             ${vehicle_info['base_link']['zed_camera']['pitch']}
+             ${vehicle_info['base_link']['zed_camera']['yaw']}"
     />
     <parent link="base_link" />
-    <child link="zed2i_base_link" />
+    <child link="zed_camera" />
   </joint>
   <link name="rslidar"/>

Commit message: 243 add support for ls lidar (#244)
* feat : added ls lidar sensor driver
- #243

* feat : added lslidar support on launch level
- #243

* fix : No such key: 'lslidar'
- #243

* fix : x-forward coordinate system in lslidar

* chore : discarding lslidar points recording

File: vehicle_common/urdf/vehicle_description.xacro (robot description, xacro)
@@ -47,4 +47,18 @@
     <child link="rslidar" />
   </joint>
+  <link name="lslidar"/>
+  <joint name="ls_lidar_link" type="fixed">
+    <!-- <origin xyz="2.8 0 0.2" rpy="0 0 0" /> -->
+    <origin
+        xyz="${vehicle_info['base_link']['lslidar']['x']}
+             ${vehicle_info['base_link']['lslidar']['y']}
+             ${vehicle_info['base_link']['lslidar']['z']}"
+        rpy="${vehicle_info['base_link']['lslidar']['roll']}
+             ${vehicle_info['base_link']['lslidar']['pitch']}
+             ${vehicle_info['base_link']['lslidar']['yaw']}"
+    />
+    <parent link="base_link" />
+    <child link="lslidar" />
+  </joint>
   <link name="rplidar"/>
   <joint name="2d_lidar_link" type="fixed">

Commit message: 217 add support for itops tof camera (#236)
* feat: added itops_f25 to vehicle_description
- #217 #236

File: vehicle_common/urdf/vehicle_description.xacro (robot description, xacro)
@@ -75,3 +75,17 @@
     <child link="rplidar" />
   </joint>
+  <link name="itops_f25"/>
+  <joint name="itops_f25_link" type="fixed">
+    <!-- <origin xyz="2.8 0 0.1" rpy="0 0 0" /> -->
+    <origin
+        xyz="${vehicle_info['base_link']['itops_f25']['x']}
+             ${vehicle_info['base_link']['itops_f25']['y']}
+             ${vehicle_info['base_link']['itops_f25']['z']}"
+        rpy="${vehicle_info['base_link']['itops_f25']['roll']}
+             ${vehicle_info['base_link']['itops_f25']['pitch']}
+             ${vehicle_info['base_link']['itops_f25']['yaw']}"
+    />
+    <parent link="base_link" />
+    <child link="itops_f25" />
+  </joint>
 </robot>
